Commit message: works fine broooooo

File: gecko_description/urdf/gecko.xacro (robot description, xacro)
@@ -10,5 +10,5 @@
   </gazebo>
   <!--////////////////////////// properties ////////////////////////////////////////////////-->
-  <xacro:property name="mass" value="1" />
+  <xacro:property name="mass" value="10" />
   <!--////////////////////////// macros ////////////////////////////////////////////////-->
     <xacro:macro name="default_inertial">
@@ -299,8 +299,8 @@
     <type>transmission_interface/SimpleTransmission</type>
     <joint name="upper_left_bar_1_joint">
-      <hardwareInterface>hardware_interface/EffortJointInterface</hardwareInterface>
+      <hardwareInterface>hardware_interface/PositionJointInterface</hardwareInterface>
     </joint>
     <actuator name="motor_upper_left_bar_1_joint">
-      <hardwareInterface>hardware_interface/EffortJointInterface</hardwareInterface>
+      <hardwareInterface>hardware_interface/PositionJointInterface</hardwareInterface>
       <mechanicalReduction>1</mechanicalReduction>
     </actuator>
@@ -309,8 +309,8 @@
     <type>transmission_interface/SimpleTransmission</type>
     <joint name="upper_right_bar_1_joint">
-      <hardwareInterface>hardware_interface/EffortJointInterface</hardwareInterface>
+      <hardwareInterface>hardware_interface/PositionJointInterface</hardwareInterface>
     </joint>
     <actuator name="motor_upper_right_bar_1_joint">
-      <hardwareInterface>hardware_interface/EffortJointInterface</hardwareInterface>
+      <hardwareInterface>hardware_interface/PositionJointInterface</hardwareInterface>
       <mechanicalReduction>1</mechanicalReduction>
     </actuator>
@@ -319,8 +319,8 @@
     <type>transmission_interface/SimpleTransmission</type>
     <joint name="lower_left_bar_1_joint">
-      <hardwareInterface>hardware_interface/EffortJointInterface</hardwareInterface>
+      <hardwareInterface>hardware_interface/PositionJointInterface</hardwareInterface>
     </joint>
     <actuator name="motor_lower_left_bar_1_joint">
-      <hardwareInterface>hardware_interface/EffortJointInterface</hardwareInterface>
+      <hardwareInterface>hardware_interface/PositionJointInterface</hardwareInterface>
       <mechanicalReduction>1</mechanicalReduction>
     </actuator>
@@ -329,8 +329,8 @@
     <type>transmission_interface/SimpleTransmission</type>
     <joint name="lower_right_bar_1_joint">
-      <hardwareInterface>hardware_interface/EffortJointInterface</hardwareInterface>
+      <hardwareInterface>hardware_interface/PositionJointInterface</hardwareInterface>
     </joint>
     <actuator name="motor_lower_right_bar_1_joint">
-      <hardwareInterface>hardware_interface/EffortJointInterface</hardwareInterface>
+      <hardwareInterface>hardware_interface/PositionJointInterface</hardwareInterface>
       <mechanicalReduction>1</mechanicalReduction>
     </actuator>

Commit message: model updated

File: gecko_description/urdf/gecko.xacro (robot description, xacro)
@@ -2,4 +2,5 @@
 <robot name="gecko" xmlns:xacro="http://www.ros.org/wiki/xacro">
   <xacro:include filename="$(find gecko_description)/urdf/materials.xacro" />
+  <xacro:include filename="$(find gecko_description)/urdf/gecko.gazebo" />
     <!--////////////////////////// plugins ////////////////////////////////////////////////-->
     <gazebo>
@@ -10,9 +11,10 @@
   </gazebo>
   <!--////////////////////////// properties ////////////////////////////////////////////////-->
-  <xacro:property name="mass" value="10" />
+  <xacro:property name="high_mass" value="5" />
+  <xacro:property name="low_mass" value="0.01" />
   <!--////////////////////////// macros ////////////////////////////////////////////////-->
-    <xacro:macro name="default_inertial">
+    <xacro:macro name="default_high_inertial">
         <inertial>
-                <mass value="${mass}" />
+                <mass value="${high_mass}" />
                 <inertia ixx="1.0" ixy="0.0" ixz="0.0"
                      iyy="1.0" iyz="0.0"
@@ -20,4 +22,33 @@
         </inertial>
     </xacro:macro>
+   <xacro:macro name="default_low_inertial">
+        <inertial>
+                <mass value="${low_mass}" />
+                <inertia ixx="1.0" ixy="0.0" ixz="0.0"
+                     iyy="1.0" iyz="0.0"
+                     izz="1.0" />
+        </inertial>
+    </xacro:macro>
+    <xacro:macro name="tire">
+	<visual>
+      <geometry>
+        <cylinder length="0.1" radius="0.1"/>
+      </geometry>
+      <origin rpy="0 0 0" xyz="0 0 -0.09"/>
+      <material name="black"/>
+    </visual>
+    <collision>
+    <geometry>
+        <cylinder length="0.1" radius="0.1"/>
+      </geometry>
+      <origin rpy="0 0 0" xyz="0 0 -0.09"/>
+      <material name="red"/>
+          <surface>
+        <friction>
+          <ode><mu>100000.0</mu><mu2>100000.0</mu2></ode>
+        </friction>
+      </surface>
+      </collision>
+    </xacro:macro>
   <!--////////////////////////// left upper links ////////////////////////////////////////////////-->
   <link name="base_link">
@@ -38,5 +69,5 @@
       <material name="red"/>
       </collision>
-    <xacro:default_inertial />
+    <xacro:default_low_inertial />
   </link>
   <joint name="left_leg_joint" type="fixed">
@@ -60,5 +91,5 @@
       <material name="red"/>
           </collision>
-    <xacro:default_inertial />
+    <xacro:default_low_inertial />
   </link>
   <joint name="upper_left_bar_1_joint" type="continuous">
@@ -83,5 +114,5 @@
       <material name="red"/>
       </collision>
-    <xacro:default_inertial />
+    <xacro:default_low_inertial />
   </link>
   <joint name="upper_left_bar_2_joint" type="fixed">
@@ -106,5 +137,5 @@
       <material name="red"/>
       </collision>
-    <xacro:default_inertial />
+    <xacro:default_low_inertial />
   </link>
   <joint name="right_leg_joint" type="fixed">
@@ -128,5 +159,5 @@
       <material name="red"/>
           </collision>
-    <xacro:default_inertial />
+    <xacro:default_low_inertial />
   </link>
   <joint name="upper_right_bar_1_joint" type="continuous">
@@ -141,5 +172,5 @@
         <box size="0.05 0.2 0.05"/>
       </geometry>
-      <origin rpy="0 0 0" xyz="0 0.075 0"/>
+      <origin rpy="0 0 0" xyz="0 -0.075 0"/>
       <material name="white"/>
     </visual>
@@ -148,13 +179,13 @@
       <box size="0.05 0.2 0.05"/>
       </geometry>
-      <origin rpy="0 0 0" xyz="0 0.075 0"/>
-      <material name="red"/>
-      </collision>
-    <xacro:default_inertial />
+      <origin rpy="0 0 0" xyz="0 -0.075 0"/>
+      <material name="red"/>
+      </collision>
+    <xacro:default_low_inertial />
   </link>
   <joint name="upper_right_bar_2_joint" type="fixed">
-    <parent link="upper_right_bar_1"/>
+    <parent link="upper_bar"/>
     <child link="upper_right_bar_2"/>
-    <origin xyz="0.16 0 0"/>
+    <origin xyz="-0.78 0 0"/>
   </joint>
  <!--////////////////////////// left lower links ////////////////////////////////////////////////-->
@@ -174,5 +205,5 @@
       <material name="red"/>
           </collision>
-    <xacro:default_inertial />
+    <xacro:default_low_inertial />
   </link>
   <joint name="lower_left_bar_1_joint" type="continuous">
@@ -197,5 +228,5 @@
       <material name="red"/>
       </collision>
-    <xacro:default_inertial />
+    <xacro:default_low_inertial />
   </link>
   <joint name="lower_left_bar_2_joint" type="fixed">
@@ -220,5 +251,5 @@
       <material name="red"/>
           </collision>
-    <xacro:default_inertial />
+    <xacro:default_low_inertial />
   </link>
   <joint name="lower_right_bar_1_joint" type="continuous">
@@ -233,5 +264,5 @@
         <box size="0.05 0.2 0.05"/>
       </geometry>
-      <origin rpy="0 0 0" xyz="0 0.075 0"/>
+      <origin rpy="0 0 0" xyz="0 -0.075 0"/>
       <material name="white"/>
     </visual>
@@ -240,13 +271,13 @@
       <box size="0.05 0.2 0.05"/>
       </geometry>
-      <origin rpy="0 0 0" xyz="0 0.075 0"/>
-      <material name="red"/>
-      </collision>
-    <xacro:default_inertial />
+      <origin rpy="0 0 0" xyz="0 -0.075 0"/>
+      <material name="red"/>
+      </collision>
+    <xacro:default_low_inertial />
   </link>
   <joint name="lower_right_bar_2_joint" type="fixed">
-    <parent link="lower_right_bar_1"/>
+    <parent link="lower_bar"/>
     <child link="lower_right_bar_2"/>
-    <origin xyz="0.16 0 0"/>
+    <origin xyz="-0.78 0 0"/>
   </joint>
 <!-- /////////////// upper and lower fixed bars ///////////////////////////////////////-->
@@ -266,5 +297,5 @@
       <material name="red"/>
       </collision>
-    <xacro:default_inertial />
+    <xacro:default_high_inertial />
   </link>
   <joint name="upper_bar_joint" type="fixed">
@@ -288,5 +319,5 @@
       <material name="red"/>
       </collision>
-    <xacro:default_inertial />
+    <xacro:default_high_inertial />
   </link>
   <joint name="lower_bar_joint" type="fixed">
@@ -294,4 +325,77 @@
     <child link="lower_bar"/>
     <origin xyz="0 0.15 0"/>
+    </joint>
+    <!-- /////////////// 4+4 tires ///////////////////////////////////////-->
+<link name="upper_left_cylinder">
+    <xacro:tire/>
+    <xacro:default_low_inertial />
+ </link>
+   <joint name="upper_left_cylinder_joint" type="fixed">
+    <parent link="left_leg"/>
+    <child link="upper_left_cylinder"/>
+    <origin xyz="0 -0.58 0"/>
+    </joint>
+  <link name="upper_right_cylinder">
+    <xacro:tire/>
+    <xacro:default_low_inertial />
+ </link>
+   <joint name="upper_right_cylinder_joint" type="fixed">
+    <parent link="right_leg"/>
+    <child link="upper_right_cylinder"/>
+    <origin xyz="0 -0.58 0"/>
+    </joint>
+<link name="lower_left_cylinder">
+    <xacro:tire/>
+    <xacro:default_low_inertial />
+ </link>
+   <joint name="lower_left_cylinder_joint" type="fixed">
+    <parent link="left_leg"/>
+    <child link="lower_left_cylinder"/>
+    <origin xyz="0 0.58 0"/>
+    </joint>
+<link name="lower_right_cylinder">
+    <xacro:tire/>
+    <xacro:default_low_inertial />
+ </link>
+   <joint name="lower_right_cylinder_joint" type="fixed">
+    <parent link="right_leg"/>
+    <child link="lower_right_cylinder"/>
+    <origin xyz="0 0.58 0"/>
+    </joint>
+  <link name="upper_left_inside_cylinder">
+    <xacro:tire/>
+    <xacro:default_high_inertial />
+ </link>
+   <joint name="upper_left_inside_cylinder_joint" type="continuous">
+    <parent link="upper_bar"/>
+    <child link="upper_left_inside_cylinder"/>
+    <origin xyz="-0.15 0 0"/>
+    </joint>
+  <link name="upper_right_inside_cylinder">
+    <xacro:tire/>
+    <xacro:default_high_inertial />
+ </link>
+   <joint name="upper_right_inside_cylinder_joint" type="continuous">
+    <parent link="upper_bar"/>
+    <child link="upper_right_inside_cylinder"/>
+    <origin xyz="-0.6 0 0"/>
+    </joint>
+  <link name="lower_left_inside_cylinder">
+    <xacro:tire/>
+    <xacro:default_high_inertial />
+ </link>
+   <joint name="lower_left_inside_cylinder_joint" type="continuous">
+    <parent link="lower_bar"/>
+    <child link="lower_left_inside_cylinder"/>
+    <origin xyz="-0.15 0 0"/>
+    </joint>
+  <link name="lower_right_inside_cylinder">
+    <xacro:tire/>
+    <xacro:default_high_inertial />
+ </link>
+   <joint name="lower_right_inside_cylinder_joint" type="continuous">
+    <parent link="lower_bar"/>
+    <child link="lower_right_inside_cylinder"/>
+    <origin xyz="-0.6 0 0"/>
     </joint>
 <!-- /////////////// transmissions ///////////////////////////////////////-->

Commit message: upated friction factor

File: gecko_description/urdf/gecko.xacro (robot description, xacro)
@@ -12,5 +12,5 @@
   <!--////////////////////////// properties ////////////////////////////////////////////////-->
   <xacro:property name="high_mass" value="5" />
-  <xacro:property name="low_mass" value="0.01" />
+  <xacro:property name="low_mass" value="5" />
   <!--////////////////////////// macros ////////////////////////////////////////////////-->
     <xacro:macro name="default_high_inertial">
